File: PCB/Phizard_2_0_5.kicad_pcb (KiCad board)
At the start: 2 copper layers, 125.5 x 90.3 mm, 129 parts, among them J1 Conn_01x06_Female, J10 Conn_01x02, J11 Conn_01x02, J12 USB_C_Receptacle, J14 Conn_01x06, J15 Conn_01x06, J2 Conn_01x02, J4 Conn_01x01, J5 Rumble, J6 Conn_01x06, J7 Rumble 3.3V coin motor, J8 Conn_01x07, J9 USB_C_Receptacle_USB2.0, Q1 Q_NMOS_GSD, Q2 Q_PMOS_GDS, Q3 Q_NMOS_GSD, SW1 A, SW10 Dup, SW11 Dright, SW12 Ddown, SW2 B, SW3 X, SW4 Y, SW5 Start, SW6 L, SW7 R, SW8 Z, SW9 Dleft, U1 MCP3202, U10 DRV5055A3xDBZxQ1, U11 DRV5055A3xDBZxQ1, U12 USBLC6-2P6, U13 USBLC6-2P6, U2 Stickbox_Assembly_Main, U3 MCP3202, U4 DRV5055A3xDBZxQ1, U5 Stickbox_Assembly_CStick, U6 AMS1117-3.3, U7 W25Q128JVS, U8 RP2040, U9 DRV5055A3xDBZxQ1, Y1 Crystal_GND24

Commit message: Add JLCPCB production files
add JLCPCB production files
bug fixes
Parts:
- R22: footprint Resistor_SMD:R_0402_1005Metric -> Resistor_SMD:R_1206_3216Metric
- R27, R28: value R -> 5.1k
- moved R22 1.52 mm to (85.0, 74.2)
- moved ? 0.50 mm to (51.1, 75.3)
- moved ? 0.50 mm to (170.2, 75.2)
- moved SW6 0.50 mm to (51.1, 73.3)
- moved SW7 0.50 mm to (170.2, 73.2)
Routing:
- net GND: track 202.9 -> 206.8 mm
- net /R: track 73.3 -> 72.8 mm
- net /Dup: track 130.7 -> 130.2 mm
