File: PCB/Phizard_2_0_5.kicad_sch (KiCad schematic)
At the start: 119 parts, among them J1 Conn_01x06_Female, J10 Conn_01x02_Socket, J11 Conn_01x02, J12 TYPE-C 24P QCHT, J14 Conn_01x06, J15 Conn_01x06, J2 Conn_01x02, J3 Conn_01x02, J4 Conn_01x01, J5 Rumble, J6 Conn_01x06, J7 Rumble 3.3V coin motor, J8 Conn_01x07_Socket, J9 G-Switch GT-USB-7010ANS, Q1 Q_NMOS_GSD, Q2 Q_PMOS_GDS, Q3 Q_NMOS_GSD, SW1 A, SW10 Dup, SW11 Dright, SW12 Ddown, SW2 B, SW3 X, SW4 Y, SW5 Start, SW6 L, SW7 R, SW8 Z, SW9 Dleft, U1 MCP3202, U10 GH39FKSW, U11 GH39FKSW, U12 USBLC6-2P6, U13 USBLC6-2P6, U2 Stickbox_Assembly_Main, U3 MCP3202, U4 GH39FKSW, U5 Stickbox_Assembly_CStick, U6 AMS1117-3.3, U7 W25Q128JVS, U8 RP2040, U9 GH39FKSW, Y1 Crystal_GND24

Commit message: Add JLCPCB production files
add JLCPCB production files
bug fixes
Parts:
- J1, J10, J5, J7, J8: now left out of the parts list
- J9: value G-Switch GT-USB-7010ANS -> GT-USB-7010AB; LCSC C5362631 -> C963412
- R22: footprint Resistor_SMD:R_0402_1005Metric -> Resistor_SMD:R_1206_3216Metric; LCSC (none) -> C2845146
- U10, U11, U4, U9: LCSC C266230 -> C266128
